File: Circuit/Eagle/CheckBatteryVoltage.brd (EAGLE design)
At the start: 100.3 x 69.8 mm, 37 parts

Commit message: .
Parts:
- moved E$19 58.8 mm to (97.8, 60.3)
- moved E$13 58.8 mm to (97.8, 66.7)
- moved E$6 58.8 mm to (97.8, 63.5)
- moved E$16 58.8 mm to (94.6, 60.3)
- moved E$24 58.8 mm to (94.6, 66.7)
- moved E$5 19.7 mm to (64.1, 22.9)
- moved E$3 15.9 mm to (64.1, 27.9)
Other:
- board text added: "Gnd cell battery"
- board text added: "Vcc cell battery"
Changed lines of the file:
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@@
 <board>
 <plain>
-<wire x1="0" y1="0" x2="0" y2="22.86" width="1.016" layer="20"/>
-<wire x1="0" y1="22.86" x2="0" y2="41.275" width="1.016" layer="20"/>
-<wire x1="0" y1="41.275" x2="0" y2="48.26" width="1.016" layer="20"/>
-<wire x1="0" y1="48.26" x2="0" y2="69.85" width="1.016" layer="20"/>
-<wire x1="0" y1="69.85" x2="24.13" y2="69.85" width="1.016" layer="20"/>
-<wire x1="24.13" y1="69.85" x2="100" y2="69.85" width="1.016" layer="20"/>
+<wire x1="0" y1="0" x2="0" y2="22.86" width="0.508" layer="20"/>
+<wire x1="0" y1="22.86" x2="0" y2="41.275" width="0.508" layer="20"/>
+<wire x1="0" y1="41.275" x2="0" y2="48.26" width="0.508" layer="20"/>
+<wire x1="0" y1="48.26" x2="0" y2="69.85" width="0.508" layer="20"/>
+<wire x1="0" y1="69.85" x2="24.13" y2="69.85" width="0.508" layer="20"/>
+<wire x1="24.13" y1="69.85" x2="100" y2="69.85" width="0.508" layer="20"/>
 <wire x1="0" y1="0" x2="100.33" y2="0" width="0.4064" layer="20"/>
 <wire x1="100.33" y1="0" x2="100.33" y2="69.85" width="0.4064" layer="20"/>
@@
 <text x="7.62" y="65.405" size="1.016" layer="38" rot="R180">Vcc battery</text>
 <text x="90.17" y="39.37" size="1.016" layer="38">Vcc battery</text>
-<hole x="1.905" y="67.945" drill="0.35"/>
-<hole x="1.905" y="50.8" drill="0.35"/>
-<hole x="22.225" y="50.8" drill="0.35"/>
-<hole x="22.225" y="67.945" drill="0.35"/>
-<wire x1="0" y1="48.26" x2="24.13" y2="48.26" width="1.016" layer="20"/>
-<wire x1="24.13" y1="48.26" x2="24.13" y2="69.85" width="1.016" layer="20"/>
+<hole x="1.905" y="67.945" drill="2"/>
+<hole x="1.905" y="50.165" drill="2"/>
+<hole x="22.225" y="50.165" drill="2"/>
+<hole x="22.225" y="67.945" drill="2"/>
+<wire x1="0" y1="48.26" x2="24.13" y2="48.26" width="0.508" layer="20"/>
+<wire x1="24.13" y1="48.26" x2="24.13" y2="69.85" width="0.508" layer="20"/>
 <text x="8.89" y="52.07" size="1.016" layer="38" rot="R180">Tx</text>
 <dimension x1="0" y1="69.85" x2="24.13" y2="69.85" x3="12.065" y3="74.93" textsize="1.778" layer="20"/>
 <dimension x1="0" y1="48.26" x2="0" y2="69.85" x3="-7.62" y3="59.055" textsize="1.778" layer="20"/>
-<text x="8.89" y="31.75" size="1.016" layer="38" rot="R180">Gnd battery</text>
-<text x="10.795" y="37.465" size="1.016" layer="38" rot="R180">Vcc battery</text>
-<hole x="1.905" y="38.735" drill="0.35"/>
-<hole x="1.905" y="25.4" drill="0.35"/>
-<hole x="48.26" y="25.4" drill="0.35"/>
+<text x="10.16" y="31.75" size="1.016" layer="38" rot="R180">Gnd cell battery</text>
+<text x="10.16" y="37.465" size="1.016" layer="38" rot="R180">Vcc cell battery</text>
+<hole x="1.905" y="39.37" drill="2"/>
+<hole x="1.905" y="24.765" drill="2"/>
+<hole x="48.26" y="24.765" drill="2"/>
 <text x="13.97" y="25.4" size="1.016" layer="38" rot="R180">Tx</text>
-<wire x1="0" y1="41.275" x2="50.165" y2="41.275" width="1.016" layer="20"/>
-<wire x1="50.165" y1="41.275" x2="50.165" y2="22.86" width="1.016" layer="20"/>
-<wire x1="50.165" y1="22.86" x2="0" y2="22.86" width="1.016" layer="20"/>
+<wire x1="0" y1="41.275" x2="50.165" y2="41.275" width="0.508" layer="20"/>
+<wire x1="50.165" y1="41.275" x2="50.165" y2="22.86" width="0.508" layer="20"/>
+<wire x1="50.165" y1="22.86" x2="0" y2="22.86" width="0.508" layer="20"/>
 <text x="50.165" y="59.055" size="0.8128" layer="22">AVR TRASMITTER
 </text>
 <text x="74.295" y="60.325" size="0.8128" layer="22">AVR RECEIVER</text>
-<text x="43.18" y="36.83" size="0.8128" layer="22">Vcc
+<text x="41.91" y="36.195" size="0.8128" layer="22">Vcc
 </text>
-<text x="43.815" y="24.765" size="0.8128" layer="22">Gnd</text>
+<text x="41.91" y="25.4" size="0.8128" layer="22">Gnd</text>
 <text x="43.815" y="28.575" size="0.8128" layer="22">Demux
 </text>
 <text x="63.5" y="59.69" size="0.8128" layer="22">Decoupler</text>
-<hole x="48.26" y="38.735" drill="0.35"/>
+<hole x="48.26" y="39.37" drill="2"/>
 <hole x="82.55" y="42.545" drill="0.35"/>
 <hole x="83.185" y="62.865" drill="0.35"/>
@@
 <attribute name="VALUE" x="20.4724" y="60.0456" size="0.9906" layer="27" ratio="10" rot="R270"/>
 </element>
-<element name="E$3" library="discrete" library_urn="urn:adsk.eagle:library:211" package="PAD-01" package3d_urn="urn:adsk.eagle:package:12928/1" value="" x="80.01" y="26.67" smashed="yes">
-<attribute name="NAME" x="78.74" y="29.718" size="1.27" layer="25" ratio="10"/>
-<attribute name="VALUE" x="78.74" y="28.194" size="1.27" layer="27" ratio="10"/>
-</element>
-<element name="E$5" library="discrete" library_urn="urn:adsk.eagle:library:211" package="PAD-01" package3d_urn="urn:adsk.eagle:package:12928/1" value="" x="83.82" y="22.86" smashed="yes">
-<attribute name="NAME" x="82.55" y="25.908" size="1.27" layer="25" ratio="10"/>
-<attribute name="VALUE" x="82.55" y="24.384" size="1.27" layer="27" ratio="10"/>
-</element>
-<element name="E$6" library="discrete" library_urn="urn:adsk.eagle:library:211" package="PAD-01" package3d_urn="urn:adsk.eagle:package:12928/1" value="" x="71.755" y="10.795" smashed="yes">
-<attribute name="NAME" x="70.485" y="13.843" size="1.27" layer="25" ratio="10"/>
-<attribute name="VALUE" x="70.485" y="12.319" size="1.27" layer="27" ratio="10"/>
-</element>
-<element name="E$13" library="discrete" library_urn="urn:adsk.eagle:library:211" package="PAD-01" package3d_urn="urn:adsk.eagle:package:12928/1" value="" x="71.755" y="13.97" smashed="yes">
-<attribute name="NAME" x="70.485" y="17.018" size="1.27" layer="25" ratio="10"/>
-<attribute name="VALUE" x="70.485" y="15.494" size="1.27" layer="27" ratio="10"/>
-</element>
-<element name="E$24" library="discrete" library_urn="urn:adsk.eagle:library:211" package="PAD-01" package3d_urn="urn:adsk.eagle:package:12928/1" value="" x="68.58" y="13.97" smashed="yes">
-<attribute name="NAME" x="67.31" y="17.018" size="1.27" layer="25" ratio="10"/>
-<attribute name="VALUE" x="67.31" y="15.494" size="1.27" layer="27" ratio="10"/>
-</element>
-<element name="E$16" library="solpad" library_urn="urn:adsk.eagle:library:364" package="LSP10" package3d_urn="urn:adsk.eagle:package:26501/1" value="1M" x="68.58" y="7.62" smashed="yes">
-<attribute name="NAME" x="67.31" y="8.89" size="1.27" layer="25" ratio="10"/>
-<attribute name="VALUE" x="68.58" y="7.874" size="0.0254" layer="27"/>
-</element>
-<element name="E$19" library="solpad" library_urn="urn:adsk.eagle:library:364" package="LSP10" package3d_urn="urn:adsk.eagle:package:26501/1" value="" x="71.755" y="7.62" smashed="yes">
-<attribute name="NAME" x="70.485" y="8.89" size="1.27" layer="25" ratio="10"/>
-<attribute name="VALUE" x="71.755" y="7.874" size="0.0254" layer="27"/>
+<element name="E$3" library="discrete" library_urn="urn:adsk.eagle:library:211" package="PAD-01" package3d_urn="urn:adsk.eagle:package:12928/1" value="" x="64.135" y="27.94" smashed="yes">
+<attribute name="NAME" x="62.865" y="30.988" size="1.27" layer="25" ratio="10"/>
+<attribute name="VALUE" x="62.865" y="29.464" size="1.27" layer="27" ratio="10"/>
+</element>
+<element name="E$5" library="discrete" library_urn="urn:adsk.eagle:library:211" package="PAD-01" package3d_urn="urn:adsk.eagle:package:12928/1" value="" x="64.135" y="22.86" smashed="yes">
+<attribute name="NAME" x="62.865" y="25.908" size="1.27" layer="25" ratio="10"/>
+<attribute name="VALUE" x="62.865" y="24.384" size="1.27" layer="27" ratio="10"/>
+</element>
+<element name="E$6" library="discrete" library_urn="urn:adsk.eagle:library:211" package="PAD-01" package3d_urn="urn:adsk.eagle:package:12928/1" value="" x="97.79" y="63.5" smashed="yes">
+<attribute name="NAME" x="96.52" y="66.548" size="1.27" layer="25" ratio="10"/>
+<attribute name="VALUE" x="96.52" y="65.024" size="1.27" layer="27" ratio="10"/>
+</element>
+<element name="E$13" library="discrete" library_urn="urn:adsk.eagle:library:211" package="PAD-01" package3d_urn="urn:adsk.eagle:package:12928/1" value="" x="97.79" y="66.675" smashed="yes">
+<attribute name="NAME" x="96.52" y="69.723" size="1.27" layer="25" ratio="10"/>
+<attribute name="VALUE" x="96.52" y="68.199" size="1.27" layer="27" ratio="10"/>
+</element>
+<element name="E$24" library="discrete" library_urn="urn:adsk.eagle:library:211" package="PAD-01" package3d_urn="urn:adsk.eagle:package:12928/1" value="" x="94.615" y="66.675" smashed="yes">
+<attribute name="NAME" x="93.345" y="69.723" size="1.27" layer="25" ratio="10"/>
+<attribute name="VALUE" x="93.345" y="68.199" size="1.27" layer="27" ratio="10"/>
+</element>
+<element name="E$16" library="solpad" library_urn="urn:adsk.eagle:library:364" package="LSP10" package3d_urn="urn:adsk.eagle:package:26501/1" value="1M" x="94.615" y="60.325" smashed="yes">
+<attribute name="NAME" x="93.345" y="61.595" size="1.27" layer="25" ratio="10"/>
+<attribute name="VALUE" x="94.615" y="60.579" size="0.0254" layer="27"/>
+</element>
+<element name="E$19" library="solpad" library_urn="urn:adsk.eagle:library:364" package="LSP10" package3d_urn="urn:adsk.eagle:package:26501/1" value="" x="97.79" y="60.325" smashed="yes">
+<attribute name="NAME" x="96.52" y="61.595" size="1.27" layer="25" ratio="10"/>
+<attribute name="VALUE" x="97.79" y="60.579" size="0.0254" layer="27"/>
 </element>
 <element name="E$9" library="testpad" library_urn="urn:adsk.eagle:library:385" package="P1-17Y" package3d_urn="urn:adsk.eagle:package:27953/1" value="" x="89.535" y="12.7" smashed="yes">
@@
 <element name="E$14" library="ref-packages-longpad" library_urn="urn:adsk.eagle:library:337" package="ZDIO-7.5" value="zener 2.4" x="22.225" y="31.75" smashed="yes" rot="R270">
 <attribute name="NAME" x="23.9268" y="34.2392" size="1.27" layer="25" ratio="10" rot="R270"/>
-<attribute name="VALUE" x="19.685" y="36.957" size="1.27" layer="27" ratio="10"/>
+<attribute name="VALUE" x="20.32" y="36.957" size="1.27" layer="27" ratio="10"/>
 </element>
 <element name="E$15" library="eagle-ltspice" package="0204/7" value="220" x="25.4" y="31.75" smashed="yes" rot="R270">
