File: Circuit/Eagle/NanoDemultiplexerAndSDcard.brd (EAGLE design)
At the start: 100.3 x 70 mm, 16 parts

Commit message: .
Parts:
- added E$1, E$2, E$5: (no value), con-lstb:MA08-1
- added E$10, E$12, E$13, E$14, E$20, E$21, E$24, E$25, E$27, E$32, E$33, E$9: (no value), testpad:P1-13Y
- added E$11: (no value), testpad:P1-17Y
- added E$15, E$16, E$8: (no value), con-lstb:MA08-1W
- added E$19: 1000uF, ref-packages-longpad:E5-8,5
- added E$34: Attiny85, 74xx-us:DIL08
- added E$36: zener 2.4, ref-packages-longpad:ZDIO-7.5
- added E$37, E$51, E$52, E$53, E$54, E$55: (no value), solpad:LSP10
- added E$38: (no value), solpad:LSP11
- added E$39, E$42: (no value), solpad:MCS10B
- added E$40, E$43, E$46: 220, eagle-ltspice:0204/7
- added E$41, E$48, E$49, E$50, E$56, E$57, E$58, E$59, E$60, E$61, E$62, E$63, E$64, E$65, E$66, E$67, E$68: (no value), wirepad:2,54/0,8
- added E$47: Til113, ic-package:DIL06
- moved E$6 107.3 mm to (109.8, 32.0)
- moved E$3 90.4 mm to (113.6, 64.4), turned to 270 degrees
- moved E$7 14.5 mm to (20.6, 45.2)
- moved E$22 8.00 mm to (112.4, 48.0)
- moved E$30 5.23 mm to (113.2, 56.0), turned to 180 degrees
- moved E$29 1.30 mm to (106.2, 64.8)
- moved E$44 1.00 mm to (108.0, 40.4)
- moved E$45 1.00 mm to (106.2, 4.68), turned to 0 degrees
Connections:
- new net GND: E$1.6, E$1.8, E$10.TP, E$13.TP, E$19.-, E$7.P$58, E$8.5
- new net S$10: E$20.TP, E$25.TP, E$47.5
- new net S$11: E$6.A, E$6.K
- new net S$12: E$15.7, E$2.2
- new net S$13: E$15.6, E$2.3
- new net S$14: E$15.5, E$2.4
- new net S$15: E$15.4, E$2.5
- new net S$16: E$15.3, E$2.6
- new net S$17: E$15.2, E$2.7
- new net S$18: E$15.1, E$2.8
- new net S$19: E$16.8, E$5.1
- new net S$2: E$15.8, E$2.1
- new net S$20: E$16.7, E$5.2
- new net S$21: E$16.6, E$5.3
- new net S$22: E$16.5, E$5.4
- new net S$23: E$16.4, E$5.5
- new net S$24: E$16.3, E$5.6
- new net S$25: E$16.2, E$5.7
- new net S$26: E$16.1, E$5.8
- new net S$27: E$7.P$2, E$8.1
- new net S$28: E$7.P$4, E$8.2
- new net S$29: E$7.P$31, E$8.3
- new net S$3: E$1.1, E$7.P$20
- new net S$38: E$34.3, E$36.A, E$40.1
- new net S$39: E$32.TP, E$33.TP, E$34.8, E$36.C
- new net S$4: E$1.5, E$7.P$17
- new net S$40: E$34.2, E$47.1
- new net S$41: E$43.2, E$47.2
- new net S$42: E$12.TP, E$34.4, E$40.2, E$43.1
- new net S$44: E$27.TP, E$46.1, E$47.4
- new net S$45: E$21.TP, E$24.TP, E$46.2
- new net S$5: E$1.4, E$7.P$16
- new net S$7: E$1.3, E$7.P$13
- new net S$8: E$1.2, E$7.P$12
- new net S$9: E$1.7, E$14.TP, E$19.+, E$7.P$54, E$8.4, E$9.TP
Routing:
- net S$2: track 131.4 -> 4.33 mm
- net S$9: track 0.00 -> 112.5 mm
- net GND: track 0.00 -> 109.4 mm
- net S$3: track 0.00 -> 37.2 mm
- net S$42: track 0.00 -> 32.5 mm
- net S$40: track 0.00 -> 23.6 mm
- net S$29: track 0.00 -> 23.2 mm
- net S$39: track 0.00 -> 22.6 mm
- net S$5: track 0.00 -> 20.3 mm
- net S$4: track 0.00 -> 20.3 mm
- net S$7: track 0.00 -> 20.3 mm
- net S$8: track 0.00 -> 20.2 mm
- net S$38: track 0.00 -> 18.5 mm
- net S$10: track 0.00 -> 15.0 mm
- net S$41: track 0.00 -> 9.98 mm
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Other:
- board size 100.3 x 70 mm -> 100 x 70 mm
- board text added: "Demultiplexer"
- board text added: "Demux"
- board text added: "Gnd"
- board text added: "Gnd battery"
- board text added: "SD CARD"
- board text added: "SD card"
- board text added: "Tx"
- board text added: "Vcc"
- board text added: "Vcc battery"
- board text added: "gnd"
- board text added: "vcc"

Commit message: .
Connections:
- net S$39 renamed B+
- net S$42 renamed B-
- removed net S$10: E$20.TP, E$25.TP, E$47.5
- removed net S$45: E$21.TP, E$24.TP, E$46.2
- removed net S$9: E$1.7, E$14.TP, E$19.+, E$7.P$54, E$8.4, E$9.TP
- new net 5V: E$1.7, E$14.TP, E$19.+, E$20.TP, E$25.TP, E$47.5, E$7.P$54, E$8.4, E$9.TP
- net GND: now also E$21.TP, E$24.TP, E$46.2
Routing:
- net 5V: track 0.00 -> 126.8 mm
- net S$9: track 112.5 -> 0.00 mm
- net S$10: track 15.0 -> 0.00 mm
- net GND: track 109.4 -> 118.6 mm
- net S$45: track 8.98 -> 0.00 mm
Changed lines of the file:
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@@
 <setting verticaltext="up"/>
 </settings>
-<grid distance="0.1" unitdist="mm" unit="mm" style="lines" multiple="1" display="yes" altdistance="5" altunitdist="mil" altunit="mm"/>
+<grid distance="0.5" unitdist="mm" unit="mm" style="lines" multiple="1" display="yes" altdistance="5" altunitdist="mil" altunit="mm"/>
 <layers>
 <layer number="1" name="Top" color="4" fill="1" visible="yes" active="yes"/>
@@
 <layer number="19" name="Unrouted" color="6" fill="1" visible="no" active="yes"/>
 <layer number="20" name="Dimension" color="15" fill="1" visible="yes" active="yes"/>
-<layer number="21" name="tPlace" color="7" fill="1" visible="no" active="yes"/>
+<layer number="21" name="tPlace" color="7" fill="1" visible="yes" active="yes"/>
 <layer number="22" name="bPlace" color="7" fill="1" visible="no" active="yes"/>
-<layer number="23" name="tOrigins" color="15" fill="1" visible="no" active="yes"/>
+<layer number="23" name="tOrigins" color="15" fill="1" visible="yes" active="yes"/>
 <layer number="24" name="bOrigins" color="15" fill="1" visible="no" active="yes"/>
 <layer number="25" name="tNames" color="7" fill="1" visible="no" active="yes"/>
@@
 <layer number="45" name="Holes" color="7" fill="1" visible="no" active="yes"/>
 <layer number="46" name="Milling" color="3" fill="1" visible="no" active="yes"/>
-<layer number="47" name="Measures" color="7" fill="1" visible="no" active="yes"/>
+<layer number="47" name="Measures" color="7" fill="1" visible="yes" active="yes"/>
 <layer number="48" name="Document" color="7" fill="1" visible="no" active="yes"/>
 <layer number="49" name="Reference" color="7" fill="1" visible="no" active="yes"/>
@@
 <wire x1="42.9" y1="41.95" x2="42.9" y2="-0.05" width="0.4064" layer="22"/>
 <wire x1="42.9" y1="-0.05" x2="66.6" y2="-0.05" width="0.4064" layer="21"/>
-<dimension x1="42.9" y1="48.5" x2="0.9" y2="48.5" x3="21.9" y3="18.6" textsize="1.778" layer="47"/>
-<dimension x1="0.9" y1="48.5" x2="0.9" y2="24.8" x3="-6.9" y3="36.65" textsize="1.778" layer="47"/>
 <hole x="64.59" y="39.94" drill="2"/>
 <hole x="64.6" y="1.95" drill="2"/>
 <hole x="44.9" y="1.95" drill="2"/>
 <hole x="44.87" y="39.94" drill="2"/>
-<dimension x1="0.9" y1="24.8" x2="0.9" y2="26.8" x3="-2.6" y3="25.8" textsize="1.778" layer="47" dtype="diameter"/>
-<dimension x1="0.9" y1="24.8" x2="2.9" y2="24.8" x3="1.9" y3="22.8" textsize="1.778" layer="47" dtype="diameter"/>
-<dimension x1="0.9" y1="48.5" x2="0.9" y2="46.5" x3="5.4" y3="47.5" textsize="1.778" layer="47" dtype="diameter"/>
-<dimension x1="0.9" y1="48.5" x2="2.9" y2="48.5" x3="1.9" y3="40.3" textsize="1.778" layer="47" dtype="diameter"/>
-<dimension x1="42.9" y1="48.5" x2="40.9" y2="48.5" x3="41.9" y3="44.3" textsize="1.778" layer="47" dtype="diameter"/>
-<dimension x1="42.9" y1="48.5" x2="42.9" y2="46.5" x3="37.2" y3="47.5" textsize="1.778" layer="47" dtype="diameter"/>
-<dimension x1="42.9" y1="24.8" x2="42.9" y2="26.8" x3="38.6" y3="25.8" textsize="1.778" layer="47" dtype="diameter"/>
-<dimension x1="42.9" y1="24.8" x2="40.9" y2="24.8" x3="41.9" y3="28.4" textsize="1.778" layer="47" dtype="diameter"/>
 <wire x1="1.18" y1="16.69" x2="1.18" y2="35.09" width="0.4064" layer="21"/>
 <wire x1="1.18" y1="35.09" x2="42.18" y2="35.09" width="0.4064" layer="21"/>
@@
 <text x="111.08" y="37.4" size="1.778" layer="38" rot="R180">gnd</text>
 <text x="104.54" y="51.02" size="1.778" layer="38" rot="R180">vcc</text>
-<dimension x1="53" y1="70" x2="0" y2="70" x3="26.5" y3="76" textsize="1.778" layer="47"/>
 <dimension x1="0" y1="0" x2="0" y2="70" x3="-19" y3="35" textsize="1.778" layer="47"/>
 <hole x="2" y="68" drill="2"/>
@@
 <rectangle x1="-20.7" y1="70.8" x2="100.5" y2="94.2" layer="16"/>
 <rectangle x1="100.5" y1="-14.4" x2="121.8" y2="94.2" layer="16"/>
+<dimension x1="75.4" y1="11" x2="75.4" y2="59" x3="72.5" y3="35" textsize="1.778" layer="47"/>
+<dimension x1="75.4" y1="59" x2="93" y2="59" x3="84.2" y3="63" textsize="1.778" layer="47"/>
 </plain>
 <attributes>
@@
 <wire x1="38.48" y1="62.0004" x2="37.0618" y2="60.5822" width="0.8128" layer="16"/>
 <wire x1="35.8902" y1="37.719" x2="35.81" y2="37.56" width="0.8128" layer="16"/>
-<wire x1="47.5488" y1="66.5988" x2="47.5488" y2="64.2366" width="0.8128" layer="16"/>
+<wire x1="47.5488" y1="66.5988" x2="47.5488" y2="64.7366" width="0.8128" layer="16"/>
+<wire x1="47.5488" y1="64.7366" x2="47.5488" y2="64.2366" width="0.8128" layer="16"/>
 <wire x1="47.09" y1="67.0576" x2="47.5488" y2="66.5988" width="0.8128" layer="16"/>
 <wire x1="40.504434375" y1="67.0576" x2="47.09" y2="67.0576" width="0.8128" layer="16"/>
 <wire x1="47.5488" y1="64.2366" x2="47.625" y2="64.135" width="0.8128" layer="16"/>
 <wire x1="40.504434375" y1="67.0576" x2="38.48" y2="64.5" width="0.8128" layer="16"/>
+<contactref element="E$46" pad="2"/>
+<contactref element="E$21" pad="TP"/>
+<contactref element="E$24" pad="TP"/>
+<wire x1="88.011" y1="52.578" x2="88.011" y2="52.380965625" width="0.8128" layer="16"/>
+<wire x1="88.011" y1="52.380965625" x2="88.011" y2="48.4632" width="0.8128" layer="16"/>
+<wire x1="88.011" y1="48.4632" x2="88.19" y2="48.455" width="0.8128" layer="16"/>
+<wire x1="88.011" y1="52.380965625" x2="86.995" y2="53.34" width="0.8128" layer="16"/>
+<wire x1="88.773" y1="53.34" x2="89.535" y2="53.34" width="0.8128" layer="16"/>
+<wire x1="88.011" y1="52.578" x2="88.773" y2="53.34" width="0.8128" layer="16"/>
+<wire x1="88.011" y1="52.31116875" x2="86.995" y2="53.34" width="0.8128" layer="16"/>
+<wire x1="47.5488" y1="64.2366" x2="47.625" y2="64.135" width="0.8128" layer="16"/>
+<wire x1="47.5488" y1="64.7366" x2="47.625" y2="64.635" width="0.8128" layer="16"/>
+<wire x1="57.635" y1="66.245" x2="86.995" y2="53.34" width="0" layer="19" extent="1-1"/>
 </signal>
 <signal name="S$11">
@@
 <wire x1="88.19" y1="31.31" x2="85.9108" y2="31.31" width="0.8128" layer="16"/>
 </signal>
-<signal name="S$39">
+<signal name="B+">
 <contactref element="E$34" pad="8"/>
 <contactref element="E$36" pad="C"/>
@@
 <wire x1="80.6958" y1="37.0332" x2="80.57" y2="37.025" width="0.8128" layer="16"/>
 </signal>
-<signal name="S$42">
+<signal name="B-">
 <contactref element="E$43" pad="1"/>
 <contactref element="E$34" pad="4"/>
@@
 <wire x1="83.8962" y1="53.2638" x2="83.8124" y2="53.2638" width="0.8128" layer="16"/>
 </signal>
-<signal name="S$45">
-<contactref element="E$46" pad="2"/>
-<contactref element="E$21" pad="TP"/>
-<contactref element="E$24" pad="TP"/>
-<wire x1="88.011" y1="52.578" x2="88.011" y2="52.380965625" width="0.8128" layer="16"/>
-<wire x1="88.011" y1="52.380965625" x2="88.011" y2="48.4632" width="0.8128" layer="16"/>
-<wire x1="88.011" y1="48.4632" x2="88.19" y2="48.455" width="0.8128" layer="16"/>
-<wire x1="88.011" y1="52.380965625" x2="86.995" y2="53.34" width="0.8128" layer="16"/>
-<wire x1="88.773" y1="53.34" x2="89.535" y2="53.34" width="0.8128" layer="16"/>
-<wire x1="88.011" y1="52.578" x2="88.773" y2="53.34" width="0.8128" layer="16"/>
-<wire x1="88.011" y1="52.31116875" x2="86.995" y2="53.34" width="0.8128" layer="16"/>
-</signal>
-<signal name="S$9">
+<signal name="5V">
 <contactref element="E$8" pad="4"/>
 <contactref element="E$14" pad="TP"/>
@@
 <wire x1="30.861" y1="47.3346" x2="30.861" y2="37.719" width="0.8128" layer="16"/>
 <wire x1="34.5472" y1="51.0208" x2="30.861" y2="47.3346" width="0.8128" layer="16"/>
-<wire x1="34.5472" y1="63.784" x2="34.5472" y2="63.184" width="0.8128" layer="16"/>
+<wire x1="34.5472" y1="63.284" x2="34.5472" y2="63.184" width="0.8128" layer="16"/>
 <wire x1="34.5472" y1="63.184" x2="34.5472" y2="51.0208" width="0.8128" layer="16"/>
 <wire x1="35.8902" y1="64.4652" x2="34.609" y2="63.184" width="0.8128" layer="16"/>
 <wire x1="30.861" y1="37.719" x2="30.73" y2="37.56" width="0.8128" layer="16"/>
 <wire x1="35.8902" y1="64.4652" x2="35.94" y2="64.5" width="0.8128" layer="16"/>
-<wire x1="14.884" y1="63.784" x2="13.5" y2="62.4" width="0.8128" layer="16"/>
+<wire x1="14.384" y1="63.284" x2="13.5" y2="62.4" width="0.8128" layer="16"/>
 <wire x1="34.609" y1="63.184" x2="34.5472" y2="63.184" width="0.8128" layer="16"/>
-<wire x1="34.5472" y1="63.784" x2="14.884" y2="63.784" width="0.8128" layer="16"/>
+<wire x1="34.5472" y1="63.284" x2="14.384" y2="63.284" width="0.8128" layer="16"/>
 <wire x1="13.5" y1="62.4" x2="13.23" y2="61.094996875" width="0.8128" layer="16"/>
 <wire x1="13.23" y1="57.5" x2="13.23" y2="61.094996875" width="0.8128" layer="16"/>
@@
 <wire x1="57.8358" y1="61.2648" x2="57.635" y2="61.165" width="0.8128" layer="16"/>
 <wire x1="36.1188" y1="64.6938" x2="35.94" y2="64.5" width="0.8128" layer="16"/>
-</signal>
-<signal name="S$10">
 <contactref element="E$25" pad="TP"/>
 <contactref element="E$20" pad="TP"/>
@@
 <wire x1="78.105" y1="53.34" x2="78.09985" y2="53.3709" width="0.8128" layer="16"/>
 <wire x1="80.645" y1="53.34" x2="78.105" y2="53.34" width="0.8128" layer="16"/>
+<wire x1="57.635" y1="61.165" x2="78.09985" y2="53.3709" width="0" layer="19" extent="16-16"/>
 </signal>
 </signals>
