File: Circuit/Eagle/CheckBatteryVoltage12VoltsWithReset.brd (EAGLE design)
At the start: 100.3 x 70 mm, 103 parts

Commit message: Modificato per la stampa
Parts:
- added E$103, E$104, E$105, E$106, E$107, E$108: (no value), wirepad:1,6/0,8
- added STEP-UP-GND-OUT1, STEP-UP-GND-OUT2: (no value), wirepad:2,54/0,8
- E$1: value 220 -> Attiny85; device eagle-ltspice:0204/7 -> 74xx-us:DIL08
- E$17: device eagle-ltspice:0204/7 -> testpad:P1-13Y
- E$18: device transistor-fet:TO92- -> testpad:P1-13Y
- E$2: value Til113 -> zener 10v; device ic-package:DIL06 -> ref-packages-longpad:ZDIO-7.5
- E$20, E$21, E$24, E$25, E$73, E$74: device testpad:P1-13Y -> wirepad:2,54/0,8
- E$22: device pinhead:1X01/90 -> wirepad:2,54/0,8
- E$23: device ref-packages-longpad:E5-8,5 -> wirepad:2,54/0,8
- E$26: device con-lstb:MA04-1 -> wirepad:2,54/0,8
- E$28: device con-lstb:MA06-1 -> testpad:P1-13Y
- E$29: device con-wago-508:W237-132 -> testpad:P1-13Y
- E$3: value (none) -> 680; device testpad:P1-13Y -> eagle-ltspice:0204/7
- E$30: value (none) -> 220; device discrete:RS-2,5 -> eagle-ltspice:0204/7
- E$31: value (none) -> Til113; device pinhead:2X02/90 -> ic-package:DIL06
- E$34: value Attiny85 -> (none); device 74xx-us:DIL08 -> testpad:P1-13Y
- E$35: value (none) -> W203; device con-lstb:MA04-1 -> rcl:RTRIM3296W
- E$36: value zener 12v -> w501; device ref-packages-longpad:ZDIO-7.5 -> rcl:RTRIM3296W
- E$38, E$92: value (none) -> zener 4.3v; device solpad:LSP10 -> ref-packages-longpad:ZDIO-7.5
- E$39, E$93: value (none) -> 100; device solpad:LSP10 -> eagle-ltspice:0204/7
- E$4: value (none) -> 220; device switch:TL1105 -> eagle-ltspice:0204/7
- E$40: value 1k -> (none); device eagle-ltspice:0204/7 -> wirepad:1,6/0,8
- E$43: value 220 -> (none); device eagle-ltspice:0204/7 -> wirepad:1,6/0,8
- E$44: device testpad:P1-17Y -> wirepad:1,6/0,8
- E$45: device 74xx-us:DIL08 -> wirepad:1,6/0,8
- E$46: value 220 -> (none); device eagle-ltspice:0204/7 -> discrete:RS-2,5
- E$47: value Til113 -> (none); device ic-package:DIL06 -> wirepad:1,6/0,8
- E$5, E$86: value (none) -> 220; device solpad:LSP10 -> eagle-ltspice:0204/7
- E$50, E$52, E$94, E$95: device solpad:LSP10 -> wirepad:1,6/0,8
- E$53: value (none) -> Attiny85; device solpad:LSP10 -> 74xx-us:DIL08
- E$59: value (none) -> zener 10v; device wirepad:2,54/0,8 -> ref-packages-longpad:ZDIO-7.5
- E$6, E$66, E$87: value (none) -> Til113; device solpad:LSP10 -> ic-package:DIL06
- E$60: value (none) -> 680; device wirepad:2,54/0,8 -> eagle-ltspice:0204/7
- E$61, E$62: value (none) -> 220; device wirepad:2,54/0,8 -> eagle-ltspice:0204/7
- E$67, E$68, E$7, E$8, E$83, E$84, E$85, E$88: device solpad:LSP10 -> testpad:P1-13Y
- E$69, E$70, E$71: device wirepad:2,54/0,8 -> testpad:P1-13Y
- E$75: device solpad:LSP10 -> wirepad:2,54/0,8
- E$77, E$79: value zener 12v -> (none); device ref-packages-longpad:ZDIO-7.5 -> wirepad:2,54/0,8
- E$78: value 1k -> (none); device eagle-ltspice:0204/7 -> wirepad:2,54/0,8
- E$89: value (none) -> W203; device wirepad:1,6/0,8 -> rcl:RTRIM3296W
- E$91: value (none) -> w501; device solpad:LSP10 -> rcl:RTRIM3296W
- E$98: device wirepad:1,6/0,8 -> discrete:RS-2,5
- moved E$18 108.8 mm to (6.03, 8.90), turned to 270 degrees
- moved E$17 108.7 mm to (6.03, 6.37), turned to 270 degrees
- moved E$30 107.2 mm to (10.4, 20.1)
- moved E$35 102.3 mm to (13.1, 28.4), turned to 270 degrees
- moved E$59 100.5 mm to (94.1, 25.6), turned to 180 degrees
- moved E$31 98.1 mm to (16.1, 19.7)
- moved E$79 96.7 mm to (97.8, 29.2), turned to 0 degrees
- moved E$72 95.5 mm to (98.2, 2.23)
- moved E$45 90.3 mm to (19.8, 28.3), turned to 90 degrees
- moved E$70 88.4 mm to (94.2, 6.03), turned to 0 degrees
- moved E$78 88.0 mm to (90.2, 29.2), turned to 0 degrees
- moved E$62 87.9 mm to (90.4, 10.4), turned to 180 degrees
- moved E$4 86.9 mm to (21.9, 6.54), turned to 270 degrees
- moved E$38 84.4 mm to (23.6, 28.3), turned to 180 degrees
- moved E$44 81.3 mm to (27.4, 28.3), turned to 90 degrees
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Connections:
- removed net 0V: E$71.1, E$74.TP
- removed net 12V: E$12.TP, E$36.C, E$72.1, E$73.TP
- removed net B+: E$34.8, E$70.1
- removed net B-: E$2.5, E$34.4, E$40.2, E$43.1, E$69.1
- removed net S$28: E$34.3, E$36.A, E$40.1
- removed net S$32: E$1.1, E$21.TP, E$24.TP, E$46.2
- removed net S$40: E$34.2, E$47.1
- removed net S$41: E$43.2, E$47.2
- removed net S$44: E$27.TP, E$46.1, E$47.4
- new net 5.1V-STEP-UP1: E$1.8, E$24.1, E$31.5, E$36.3
- new net 5.1V-STEP-UP2: E$53.8, E$77.1, E$87.5, E$91.3
- new net IN-12V-BATTERY1: E$2.C, E$26.1, E$27.TP, E$29.TP
- new net IN-12V-BATTERY2: E$59.C, E$79.1, E$83.TP, E$85.TP
- new net IN-5V-FROM-NANO-SDCARD1: E$17.TP, E$6.5, E$7.TP
- new net IN-5V-FROM-NANO-SDCARD2: E$66.5, E$67.TP, E$70.TP
- new net IN-GND-BATTERY1: E$25.1, E$28.TP
- new net IN-GND-BATTERY2: E$78.1, E$84.TP
- new net IN-GND-NANO-SD-CARD1: E$12.TP, E$30.1, E$5.2, E$8.TP
- new net IN-GND-NANO-SD-CARD2: E$62.2, E$68.TP, E$69.TP, E$86.1
- new net IN-TO-RESET-ATTINY1: E$31.1, E$34.TP
- new net IN-TO-RESET-ATTINY2: E$87.1, E$88.TP
- new net OUT-SERIAL-DATA1: E$18.TP, E$5.1, E$6.4
- new net OUT-SERIAL-DATA2: E$62.1, E$66.4, E$71.TP
- new net PHOTO-DIODE1: E$4.2, E$6.2
- new net PHOTO-DIODE2: E$61.2, E$66.2
- new net S$10: E$91.2, E$93.2
- new net S$11: E$53.1, E$87.4, E$98.1
- new net S$7: E$1.1, E$31.4, E$46.1
- new net S$8: E$86.2, E$87.2
- new net STEP-UP-GND1: E$1.4, E$35.2, E$38.A, E$4.1, E$46.2, STEP-UP-GND-OUT1.1
- new net STEP-UP-GND2: E$53.4, E$61.1, E$89.2, E$92.A, E$98.2, STEP-UP-GND-OUT2.1
- new net TX-SERIAL-DATA1: E$1.2, E$6.1
- new net TX-SERIAL-DATA2: E$53.2, E$66.1
- new net VZ-ANALOG-REFERENCE1: E$1.5, E$38.C, E$39.1
- new net VZ-ANALOG-REFERENCE2: E$53.5, E$92.C, E$93.1
- new net VZ-BATTERY-LEVEL1: E$1.3, E$2.A, E$3.1
- new net VZ-BATTERY-LEVEL2: E$53.3, E$59.A, E$60.1
- net S$2: now also E$30.2, E$31.2; no longer E$2.4, E$34.1
- net S$3: now also E$3.2, E$35.3; no longer E$2.1, E$3.TP
- net S$4: now also E$36.2, E$39.2; no longer E$1.2, E$2.2
- net S$9: now also E$60.2, E$89.3; no longer E$20.TP, E$25.TP, E$47.5
Routing:
- net 5.1V-STEP-UP2: track 0.00 -> 103.2 mm
- net 5.1V-STEP-UP1: track 0.00 -> 103.2 mm
- net STEP-UP-GND2: track 0.00 -> 70.5 mm
- net STEP-UP-GND1: track 0.00 -> 70.5 mm
- net B-: track 62.0 -> 0.00 mm
- net IN-12V-BATTERY2: track 0.00 -> 56.0 mm
- net IN-12V-BATTERY1: track 0.00 -> 56.0 mm
- net S$40: track 51.0 -> 0.00 mm
- net 12V: track 43.3 -> 0.00 mm
- net IN-5V-FROM-NANO-SDCARD2: track 0.00 -> 28.7 mm
- net IN-5V-FROM-NANO-SDCARD1: track 0.00 -> 28.7 mm
- net IN-GND-BATTERY2: track 0.00 -> 27.8 mm
- net IN-GND-BATTERY1: track 0.00 -> 27.8 mm
- net B+: track 24.2 -> 0.00 mm
- net VZ-BATTERY-LEVEL2: track 0.00 -> 23.4 mm
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Other:
- outline, holes or cut-outs redrawn

Commit message: .
Parts:
- added E$109, E$110, E$111, E$112, E$113, E$114, E$115, E$116, E$117, E$118, E$119, E$120, E$125, E$126, E$127, E$128, E$130, E$131, E$132, E$133, E$134, E$135, E$136, E$137, E$138, E$139, E$140, E$141, E$142, E$143, E$144: (no value), wirepad:1,6/0,8
- added E$121: W203, rcl:RTRIM3296W
- added E$122: w501, rcl:RTRIM3296W
- added E$123: zener 4.3v, ref-packages-longpad:ZDIO-7.5
- added E$124: 100, eagle-ltspice:0204/7
- added E$129: (no value), discrete:RS-2,5
- E$106: value (none) -> 220; device wirepad:1,6/0,8 -> eagle-ltspice:0204/7
- E$107: value (none) -> Til113; device wirepad:1,6/0,8 -> ic-package:DIL06
- E$108, E$96, E$97: device wirepad:1,6/0,8 -> testpad:P1-13Y
- E$53: value Attiny85 -> (none); device 74xx-us:DIL08 -> wirepad:1,6/0,8
- E$59: value zener 10v -> (none); device ref-packages-longpad:ZDIO-7.5 -> wirepad:1,6/0,8
- E$60: value 680 -> (none); device eagle-ltspice:0204/7 -> wirepad:1,6/0,8
- E$61, E$62: value 220 -> (none); device eagle-ltspice:0204/7 -> wirepad:1,6/0,8
- E$66: value Til113 -> (none); device ic-package:DIL06 -> wirepad:1,6/0,8
- E$67, E$68, E$69, E$70, E$71: device testpad:P1-13Y -> wirepad:1,6/0,8
- E$72: device wirepad:2,54/0,8 -> wirepad:1,6/0,8
- E$73: value (none) -> Attiny85; device wirepad:2,54/0,8 -> 74xx-us:DIL08
- E$74: value (none) -> zener 10v; device wirepad:2,54/0,8 -> ref-packages-longpad:ZDIO-7.5
- E$75: value (none) -> 680; device wirepad:2,54/0,8 -> eagle-ltspice:0204/7
- E$77, E$78: value (none) -> 220; device wirepad:2,54/0,8 -> eagle-ltspice:0204/7
- E$79: value (none) -> Til113; device wirepad:2,54/0,8 -> ic-package:DIL06
- E$86: value 220 -> (none); device eagle-ltspice:0204/7 -> testpad:P1-13Y
- E$87: value Til113 -> (none); device ic-package:DIL06 -> testpad:P1-13Y
- E$88: device testpad:P1-13Y -> wirepad:2,54/0,8
- E$89: value W203 -> (none); device rcl:RTRIM3296W -> wirepad:2,54/0,8
- E$91: value w501 -> (none); device rcl:RTRIM3296W -> wirepad:2,54/0,8
- E$92: value zener 4.3v -> (none); device ref-packages-longpad:ZDIO-7.5 -> wirepad:2,54/0,8
- E$93: value 100 -> (none); device eagle-ltspice:0204/7 -> wirepad:2,54/0,8
- E$94, E$95: device wirepad:1,6/0,8 -> wirepad:2,54/0,8
- E$98: device discrete:RS-2,5 -> testpad:P1-13Y
- moved E$70 80.5 mm to (13.7, 5.00), turned to 270 degrees
- moved E$69 75.6 mm to (7.80, 5.40), turned to 270 degrees
- moved E$67 74.7 mm to (26.2, 30.5), turned to 270 degrees
- moved E$68 73.1 mm to (7.80, 8.00), turned to 270 degrees
- moved E$61 67.9 mm to (26.2, 22.8), turned to 270 degrees
- moved E$66 65.2 mm to (29.9, 30.5)
- moved E$62 61.2 mm to (29.6, 17.2), turned to 270 degrees
- moved E$72 59.3 mm to (41.4, 19.2), turned to 270 degrees
- moved E$21 55.8 mm to (49.6, 1.83), turned to 270 degrees
- moved E$22 55.6 mm to (2.38, 1.83), turned to 270 degrees
- moved E$20 55.3 mm to (49.6, 30.8), turned to 270 degrees
- moved E$23 55.2 mm to (2.38, 31.0), turned to 270 degrees
- moved E$59 52.6 mm to (41.5, 26.8), turned to 270 degrees
- moved E$71 51.5 mm to (41.4, 16.9), turned to 270 degrees
- moved E$92 51.1 mm to (98.5, 67.4), turned to 180 degrees
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Connections:
- net 5.1V-STEP-UP2: now also E$107.5, E$122.3, E$73.8, E$93.1; no longer E$53.8, E$77.1, E$87.5, E$91.3
- net IN-12V-BATTERY2: now also E$74.C, E$95.1, E$96.TP, E$98.TP; no longer E$59.C, E$79.1, E$83.TP, E$85.TP
- net IN-5V-FROM-NANO-SDCARD2: now also E$79.5, E$83.TP, E$86.TP; no longer E$66.5, E$67.TP, E$70.TP
- net IN-GND-BATTERY2: now also E$94.1, E$97.TP; no longer E$78.1, E$84.TP
- net IN-GND-NANO-SD-CARD2: now also E$106.1, E$78.2, E$84.TP, E$85.TP; no longer E$62.2, E$68.TP, E$69.TP, E$86.1
- net IN-TO-RESET-ATTINY2: now also E$107.1, E$108.TP; no longer E$87.1, E$88.TP
- net OUT-SERIAL-DATA2: now also E$78.1, E$79.4, E$87.TP; no longer E$62.1, E$66.4, E$71.TP
- net PHOTO-DIODE2: now also E$77.2, E$79.2; no longer E$61.2, E$66.2
- net S$10: now also E$122.2, E$124.2; no longer E$91.2, E$93.2
- net S$11: now also E$107.4, E$129.1, E$73.1; no longer E$53.1, E$87.4, E$98.1
- net S$8: now also E$106.2, E$107.2; no longer E$86.2, E$87.2
- net S$9: now also E$121.3, E$75.2; no longer E$60.2, E$89.3
- net STEP-UP-GND2: now also E$121.2, E$123.A, E$129.2, E$73.4, E$77.1; no longer E$53.4, E$61.1, E$89.2, E$92.A, E$98.2
- net TX-SERIAL-DATA2: now also E$73.2, E$79.1; no longer E$53.2, E$66.1
- net VZ-ANALOG-REFERENCE2: now also E$123.C, E$124.1, E$73.5; no longer E$53.5, E$92.C, E$93.1
- net VZ-BATTERY-LEVEL2: now also E$73.3, E$74.A, E$75.1; no longer E$53.3, E$59.A, E$60.1
Other:
- outline, holes or cut-outs redrawn
