File: Circuit/Eagle/NanoDemultiplexerAndSDcardNew.brd (EAGLE design)
At the start: 100 x 70 mm, 43 parts

Commit message: .
Parts:
- removed E$11, E$44: (no value), testpad:P1-17Y
- removed E$17: (no value), eagle-ltspice:0204/7
- removed E$18: (no value), transistor-fet:TO92-
- removed E$22: (no value), pinhead:1X01/90
- removed E$23: (no value), ref-packages-longpad:E5-8,5
- removed E$26, E$35: (no value), con-lstb:MA04-1
- removed E$28: (no value), con-lstb:MA06-1
- removed E$29: (no value), con-wago-508:W237-132
- removed E$3: (no value), con-lstb:MA05-1
- removed E$30: (no value), discrete:RS-2,5
- removed E$31: (no value), pinhead:2X02/90
- removed E$37: (no value), solpad:LSP10
- removed E$38: (no value), solpad:LSP11
- removed E$39: (no value), solpad:MCS10B
- removed E$4: (no value), switch:TL1105
- removed E$41, E$67, E$68: (no value), wirepad:2,54/0,8
- removed E$45: (no value), 74xx-us:DIL08
- removed E$6: (no value), led:LED3MM
Connections:
- removed net S$11: E$6.A, E$6.K
- new net S$9: E$7.P$9, E$8.5
Routing:
- net S$9: track 0.00 -> 5.87 mm
- net S$11: track 2.77 -> 0.00 mm
Other:
- board size 100 x 70 mm -> 67.5 x 70 mm
- board text added: "buzzer"
