File: Circuit/Eagle/new_era_for_AI/NanoDemultiplexerAndSDcardNew.brd (EAGLE design)
At the start: 94 x 70 mm, 18 parts

Commit message: .
Parts:
- added E$13, E$20, E$21, E$22, E$23, E$24, E$25, E$26: (no value), solpad:MCS10B
Routing:
- net 5V: track 291.8 -> 299.6 mm
