File: Circuit/Eagle/new_era_for_AI/NanoDemultiplexerAndSDcardNew3.brd (EAGLE design)
At the start: 94 x 70 mm, 22 parts

Commit message: .
Parts:
- moved E$10 4.30 mm to (62.0, 8.99)
- moved E$9 4.30 mm to (59.5, 8.99)
Routing:
- net GND: track 0.00 -> 78.6 mm
- net 5V: track 0.00 -> 68.4 mm
Changed lines of the file:
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@@
 <attribute name="VALUE" x="91.678" y="32.523" size="1.27" layer="27" ratio="10" rot="R90"/>
 </element>
-<element name="E$9" library="testpad" library_urn="urn:adsk.eagle:library:385" package="P1-13Y" package3d_urn="urn:adsk.eagle:package:27947/1" value="" x="61.97833125" y="5.487028125" smashed="yes" rot="R180">
-<attribute name="NAME" x="62.86733125" y="3.328028125" size="1.27" layer="25" ratio="10" rot="R180"/>
-<attribute name="VALUE" x="61.97833125" y="5.487028125" size="0.0254" layer="27" rot="R180"/>
+<element name="E$9" library="testpad" library_urn="urn:adsk.eagle:library:385" package="P1-13Y" package3d_urn="urn:adsk.eagle:package:27947/1" value="" x="59.47833125" y="8.987028125" smashed="yes" rot="R180">
+<attribute name="NAME" x="60.36733125" y="6.828028125" size="1.27" layer="25" ratio="10" rot="R180"/>
+<attribute name="VALUE" x="59.47833125" y="8.987028125" size="0.0254" layer="27" rot="R180"/>
 </element>
-<element name="E$10" library="testpad" library_urn="urn:adsk.eagle:library:385" package="P1-13Y" package3d_urn="urn:adsk.eagle:package:27947/1" value="" x="64.47833125" y="5.487028125" smashed="yes" rot="R180">
-<attribute name="NAME" x="65.36733125" y="3.328028125" size="1.27" layer="25" ratio="10" rot="R180"/>
-<attribute name="VALUE" x="64.47833125" y="5.487028125" size="0.0254" layer="27" rot="R180"/>
+<element name="E$10" library="testpad" library_urn="urn:adsk.eagle:library:385" package="P1-13Y" package3d_urn="urn:adsk.eagle:package:27947/1" value="" x="61.97833125" y="8.987028125" smashed="yes" rot="R180">
+<attribute name="NAME" x="62.86733125" y="6.828028125" size="1.27" layer="25" ratio="10" rot="R180"/>
+<attribute name="VALUE" x="61.97833125" y="8.987028125" size="0.0254" layer="27" rot="R180"/>
 </element>
 <element name="E$4" library="con-lsta" library_urn="urn:adsk.eagle:library:161" package="FE06W" package3d_urn="urn:adsk.eagle:package:8198/1" value="" x="55.67143125" y="22.70691875" smashed="yes" rot="R90">
@@
 <contactref element="E$16" pad="-"/>
 <contactref element="E$13" pad="-"/>
-<wire x1="69.5" y1="61.778" x2="90.65" y2="51.21" width="0" layer="19" extent="1-1"/>
-<wire x1="61.73336875" y1="68.611575" x2="69.5" y2="61.778" width="0" layer="19" extent="1-1"/>
+<wire x1="61.97833125" y1="26.52166875" x2="61.97833125" y2="8.987028125" width="1.016" layer="16"/>
+<wire x1="59.44308125" y1="29.05691875" x2="55.67143125" y2="29.05691875" width="1.016" layer="16"/>
+<wire x1="61.97833125" y1="26.52166875" x2="59.44308125" y2="29.05691875" width="1.016" layer="16"/>
+<wire x1="55.67143125" y1="29.05691875" x2="55.67143125" y2="35.89343125" width="1.016" layer="16"/>
+<wire x1="55.67143125" y1="35.89343125" x2="55.778" y2="36" width="1.016" layer="16"/>
+<wire x1="90.65" y1="51.21" x2="90.65" y2="60.35" width="1.016" layer="16"/>
+<wire x1="89.222" y1="61.778" x2="69.5" y2="61.778" width="1.016" layer="16"/>
+<wire x1="90.65" y1="60.35" x2="89.222" y2="61.778" width="1.016" layer="16"/>
+<wire x1="56" y1="55.722" x2="55.722" y2="56" width="1.016" layer="16"/>
+<wire x1="55.722" y1="56" x2="46.5" y2="56" width="1.016" layer="16"/>
+<wire x1="46.5" y1="56" x2="44.904265625" y2="54.404265625" width="1.016" layer="16"/>
+<wire x1="44.904265625" y1="54.404265625" x2="44.904265625" y2="50.436003125" width="1.016" layer="16"/>
+<wire x1="69.5" y1="61.778" x2="61.73336875" y2="68.611575" width="0" layer="19" extent="1-1"/>
 <wire x1="56" y1="55.722" x2="61.73336875" y2="68.611575" width="0" layer="19" extent="1-1"/>
-<wire x1="44.904265625" y1="50.436003125" x2="56" y2="55.722" width="0" layer="19" extent="1-1"/>
 <wire x1="55.778" y1="36" x2="44.904265625" y2="50.436003125" width="0" layer="19" extent="1-1"/>
-<wire x1="55.67143125" y1="29.05691875" x2="55.778" y2="36" width="0" layer="19" extent="1-1"/>
 <wire x1="73.559" y1="32.451" x2="55.778" y2="36" width="0" layer="19" extent="1-1"/>
-<wire x1="64.47833125" y1="5.487028125" x2="55.67143125" y2="29.05691875" width="0" layer="19" extent="1-1"/>
-<wire x1="39.7122125" y1="5.180696875" x2="64.47833125" y2="5.487028125" width="0" layer="19" extent="1-1"/>
+<wire x1="39.7122125" y1="5.180696875" x2="61.97833125" y2="8.987028125" width="0" layer="19" extent="1-1"/>
 <wire x1="13.32" y1="5.1" x2="39.7122125" y2="5.180696875" width="0" layer="19" extent="1-1"/>
 <wire x1="15.49" y1="43.7" x2="44.904265625" y2="50.436003125" width="0" layer="19" extent="1-1"/>
@@
 <contactref element="E$16" pad="+"/>
 <contactref element="E$13" pad="+"/>
+<wire x1="59.47833125" y1="26.02166875" x2="59.47833125" y2="8.987028125" width="1.016" layer="16"/>
+<wire x1="58.98308125" y1="26.51691875" x2="55.67143125" y2="26.51691875" width="1.016" layer="16"/>
+<wire x1="59.47833125" y1="26.02166875" x2="58.98308125" y2="26.51691875" width="1.016" layer="16"/>
+<wire x1="52.222" y1="36" x2="52.222" y2="27.778" width="1.016" layer="16"/>
+<wire x1="53.48308125" y1="26.51691875" x2="55.67143125" y2="26.51691875" width="1.016" layer="16"/>
+<wire x1="52.222" y1="27.778" x2="53.48308125" y2="26.51691875" width="1.016" layer="16"/>
+<wire x1="75.41" y1="51.21" x2="74" y2="52.62" width="1.016" layer="16"/>
+<wire x1="74" y1="52.62" x2="74" y2="55" width="1.016" layer="16"/>
+<wire x1="74" y1="55" x2="70.778" y2="58.222" width="1.016" layer="16"/>
+<wire x1="70.778" y1="58.222" x2="69.5" y2="58.222" width="1.016" layer="16"/>
+<wire x1="56" y1="59.278" x2="40" y2="59.278" width="1.016" layer="16"/>
+<wire x1="40" y1="59.278" x2="40" y2="50.6117375" width="1.016" layer="16"/>
+<wire x1="39.824265625" y1="50.436003125" x2="40" y2="50.6117375" width="1.016" layer="16"/>
 <wire x1="56" y1="59.278" x2="59.19336875" y2="68.611575" width="0" layer="19" extent="1-1"/>
-<wire x1="69.5" y1="58.222" x2="56" y2="59.278" width="0" layer="19" extent="1-1"/>
-<wire x1="75.41" y1="51.21" x2="69.5" y2="58.222" width="0" layer="19" extent="1-1"/>
-<wire x1="39.824265625" y1="50.436003125" x2="56" y2="59.278" width="0" layer="19" extent="1-1"/>
 <wire x1="41.9" y1="43.816528125" x2="39.824265625" y2="50.436003125" width="0" layer="19" extent="1-1"/>
 <wire x1="52.222" y1="36" x2="41.9" y2="43.816528125" width="0" layer="19" extent="1-1"/>
-<wire x1="55.67143125" y1="26.51691875" x2="52.222" y2="36" width="0" layer="19" extent="1-1"/>
+<wire x1="69.5" y1="58.222" x2="56" y2="59.278" width="0" layer="19" extent="1-1"/>
 <wire x1="73.559" y1="29.911" x2="55.67143125" y2="26.51691875" width="0" layer="19" extent="1-1"/>
-<wire x1="61.97833125" y1="5.487028125" x2="55.67143125" y2="26.51691875" width="0" layer="19" extent="1-1"/>
-<wire x1="34.6322125" y1="5.180696875" x2="61.97833125" y2="5.487028125" width="0" layer="19" extent="1-1"/>
+<wire x1="34.6322125" y1="5.180696875" x2="59.47833125" y2="8.987028125" width="0" layer="19" extent="1-1"/>
 <wire x1="18.4" y1="5.1" x2="34.6322125" y2="5.180696875" width="0" layer="19" extent="1-1"/>
 </signal>
@@
 <contactref element="E$6" pad="RX"/>
 <contactref element="E$8" pad="1"/>
-<wire x1="66.051684375" y1="49.0141875" x2="77.95" y2="51.21" width="0" layer="19" extent="1-1"/>
+<wire x1="77.95" y1="51.21" x2="66.051684375" y2="49.0141875" width="0" layer="19" extent="1-1"/>
 </signal>
 <signal name="S$10">

Commit message: .
Parts:
- added E$19, E$20, E$21: (no value), testpad:P1-13Y
- added E$22, E$23, E$25, E$26, E$29, E$30, E$31, E$32, E$33, E$34, E$35, E$36, E$37, E$38, E$39, E$40, E$41, E$42, E$43, E$44, E$45, E$46, E$47, E$48, E$49, E$50, E$51, E$52, E$53, E$54: (no value), solpad:MCS10B
- E$11: device con-molex:22-23-2021 -> testpad:P1-13Y
- moved E$24 55.1 mm to (75.5, 51.7)
- moved E$11 46.4 mm to (40.0, 67.0), turned to 180 degrees
- moved E$8 7.81 mm to (69.1, 45.2), turned to 270 degrees
- moved E$28 7.43 mm to (36.4, 38.8)
- moved E$27 6.80 mm to (26.4, 38.3)
- moved E$81 6.04 mm to (16.8, 38.2)
- moved E$17 5.32 mm to (61.4, 64.6)
- moved E$16 4.53 mm to (55.5, 53.0)
- moved E$13 3.00 mm to (69.5, 57.0)
- moved E$7 3.00 mm to (29.7, 55.1)
- moved E$12 1.12 mm to (33.6, 5.68)
- moved E$15 1.12 mm to (19.4, 5.60)
- moved E$6 0.50 mm to (84.3, 60.6)
Connections:
- new net SPK3: E$11.TP, E$7.P$24
- new net SPK4: E$21.TP, E$7.P$25
- net S0: now also E$32.MP, E$34.MP
- net S1: now also E$31.MP, E$35.MP
- net S2: now also E$30.MP, E$36.MP
- net S3: now also E$29.MP, E$37.MP
- net SPK1: now also E$19.TP; no longer E$11.1
- net SPK2: now also E$20.TP; no longer E$11.2
- net TX: now also E$25.MP, E$26.MP
Routing:
- net 5V: track 68.4 -> 384.5 mm
- net GND: track 78.6 -> 376.8 mm
- net S$10: track 0.00 -> 153.3 mm
- net SIGN: track 0.00 -> 127.2 mm
- net MOSI: track 0.00 -> 96.6 mm
- net SCK: track 0.00 -> 83.9 mm
- net MISO: track 0.00 -> 80.6 mm
- net VOLUME-CONTROL: track 0.00 -> 59.3 mm
- net S$4: track 0.00 -> 52.8 mm
- net RESET: track 0.00 -> 50.4 mm
- net S$2: track 0.00 -> 12.7 mm
- net RX: track 0.00 -> 11.3 mm
- net TX: track 0.00 -> 7.70 mm
- net S1: track 0.00 -> 6.78 mm
- net S0: track 0.00 -> 6.77 mm
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