File: Circuit/Eagle/new_era_for_AI/check_battery_interrupt_mode.brd (EAGLE design)
At the start: 51.6 x 28 mm, 29 parts

Commit message: .
Parts:
- moved E$13 0.40 mm to (19.4, 26.0)
Routing:
- net S$2: track 11.7 -> 15.6 mm
- net EXT-5V: track 13.5 -> 15.4 mm
- net VZ-BATTERY-LEVEL: track 18.8 -> 19.7 mm
- net S$7: track 59.5 -> 60.2 mm
Other:
- board text added: "check-battery-module v2.00"
- board text removed: "check-battery-module v1.00"
